File: DC Load/adcdac.kicad_sch (KiCad schematic)
At the start: 31 parts, among them U11 MAX5217, U12 ADS131M02IPWR, U13 OPA277UA, U8 OPA2182, X1 FD0810004

Commit message: Assign temporary footprints
Parts:
- C13, C14, C17, C18, C25, C26, C29, C30, C31, C32, C33, C34, C35: footprint (none) -> Capacitor_SMD:C_0201_0603Metric
- R25, R28, R29, R30, R37, R38, R42, R44, R48, R49: footprint (none) -> Resistor_SMD:R_0603_1608Metric
- RV1: footprint (none) -> Potentiometer_THT:Potentiometer_Bourns_3296Y_Vertical
- TP1, TP2: footprint (none) -> TestPoint:TestPoint_Loop_D2.50mm_Drill1.0mm
- U12: footprint SOP65P640X120-20N -> SamacSys_Parts:SOP65P640X120-20N
- U13: footprint SOIC127P600X175-8N -> SamacSys_Parts:SOIC127P600X175-8N
- U8: footprint (none) -> Package_SO:VSSOP-8_3.0x3.0mm_P0.65mm
- X1: footprint (none) -> Crystal:Crystal_SMD_3225-4Pin_3.2x2.5mm_HandSoldering
Changed lines of the file:
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@@
     (property "Reference" "U8" (id 0) (at 198.12 132.08 0))
     (property "Value" "OPA2182" (id 1) (at 207.01 120.65 0))
-    (property "Footprint" "" (id 2) (at 203.2 125.73 0)
+    (property "Footprint" "Package_SO:VSSOP-8_3.0x3.0mm_P0.65mm" (id 2) (at 203.2 125.73 0)
       (effects (font (size 1.27 1.27)) hide)
     )
@@
       (effects (font (size 1.27 1.27)) (justify right))
     )
-    (property "Footprint" "" (id 2) (at 250.698 43.18 90)
+    (property "Footprint" "Resistor_SMD:R_0603_1608Metric" (id 2) (at 250.698 43.18 90)
       (effects (font (size 1.27 1.27)) hide)
     )
@@
       (effects (font (size 1.27 1.27)) (justify right))
     )
-    (property "Footprint" "" (id 2) (at 244.348 55.88 90)
+    (property "Footprint" "Resistor_SMD:R_0603_1608Metric" (id 2) (at 244.348 55.88 90)
       (effects (font (size 1.27 1.27)) hide)
     )
@@
       (effects (font (size 1.27 1.27)) (justify left))
     )
-    (property "Footprint" "" (id 2) (at 243.84 38.1 0)
+    (property "Footprint" "TestPoint:TestPoint_Loop_D2.50mm_Drill1.0mm" (id 2) (at 243.84 38.1 0)
       (effects (font (size 1.27 1.27)) hide)
     )
@@
       (effects (font (size 1.27 1.27)) (justify right))
     )
-    (property "Footprint" "" (id 2) (at 185.928 58.42 90)
+    (property "Footprint" "Resistor_SMD:R_0603_1608Metric" (id 2) (at 185.928 58.42 90)
       (effects (font (size 1.27 1.27)) hide)
     )
@@
     (property "Reference" "X1" (id 0) (at 54.61 31.75 0))
     (property "Value" "FD0810004" (id 1) (at 55.88 44.45 0))
-    (property "Footprint" "" (id 2) (at 77.47 46.99 0)
+    (property "Footprint" "Crystal:Crystal_SMD_3225-4Pin_3.2x2.5mm_HandSoldering" (id 2) (at 77.47 46.99 0)
       (effects (font (size 1.27 1.27)) hide)
     )
@@
     (property "Reference" "U13" (id 0) (at 203.2 41.91 0))
     (property "Value" "OPA277UA" (id 1) (at 219.71 41.91 0))
-    (property "Footprint" "SOIC127P600X175-8N" (id 2) (at 166.37 46.99 0)
+    (property "Footprint" "SamacSys_Parts:SOIC127P600X175-8N" (id 2) (at 166.37 46.99 0)
       (effects (font (size 1.27 1.27)) (justify left) hide)
     )
@@
       (effects (font (size 1.27 1.27)) (justify left))
     )
-    (property "Footprint" "" (id 2) (at 160.02 180.34 0)
+    (property "Footprint" "Package_SO:VSSOP-8_3.0x3.0mm_P0.65mm" (id 2) (at 160.02 180.34 0)
       (effects (font (size 1.27 1.27)) hide)
     )
@@
       (effects (font (size 1.27 1.27)) (justify right))
     )
-    (property "Footprint" "" (id 2) (at 244.348 43.18 90)
+    (property "Footprint" "Resistor_SMD:R_0603_1608Metric" (id 2) (at 244.348 43.18 90)
       (effects (font (size 1.27 1.27)) hide)
     )
@@
     (property "Reference" "RV1" (id 0) (at 210.82 38.1 90))
     (property "Value" "20K" (id 1) (at 215.9 38.1 90))
-    (property "Footprint" "" (id 2) (at 213.36 35.56 0)
+    (property "Footprint" "Potentiometer_THT:Potentiometer_Bourns_3296Y_Vertical" (id 2) (at 213.36 35.56 0)
       (effects (font (size 1.27 1.27)) hide)
     )
@@
     (property "Reference" "R44" (id 0) (at 168.91 92.71 90))
     (property "Value" "1K" (id 1) (at 168.91 97.79 90))
-    (property "Footprint" "" (id 2) (at 168.91 97.028 90)
+    (property "Footprint" "Resistor_SMD:R_0603_1608Metric" (id 2) (at 168.91 97.028 90)
       (effects (font (size 1.27 1.27)) hide)
     )
@@
       (effects (font (size 1.27 1.27)) (justify right))
     )
-    (property "Footprint" "" (id 2) (at 37.7952 40.64 0)
+    (property "Footprint" "Capacitor_SMD:C_0201_0603Metric" (id 2) (at 37.7952 40.64 0)
       (effects (font (size 1.27 1.27)) hide)
     )
@@
     (property "Reference" "U8" (id 0) (at 147.32 129.54 0))
     (property "Value" "OPA2182" (id 1) (at 147.32 132.08 0))
-    (property "Footprint" "" (id 2) (at 147.32 138.43 0)
+    (property "Footprint" "Package_SO:VSSOP-8_3.0x3.0mm_P0.65mm" (id 2) (at 147.32 138.43 0)
       (effects (font (size 1.27 1.27)) hide)
     )
@@
       (effects (font (size 1.27 1.27)) (justify right))
     )
-    (property "Footprint" "" (id 2) (at 74.6252 45.72 0)
+    (property "Footprint" "Capacitor_SMD:C_0201_0603Metric" (id 2) (at 74.6252 45.72 0)
       (effects (font (size 1.27 1.27)) hide)
     )
@@
       (effects (font (size 1.27 1.27)) (justify left))
     )
-    (property "Footprint" "" (id 2) (at 141.9352 184.15 0)
+    (property "Footprint" "Capacitor_SMD:C_0201_0603Metric" (id 2) (at 141.9352 184.15 0)
       (effects (font (size 1.27 1.27)) hide)
     )
@@
       (effects (font (size 1.27 1.27)) (justify left))
     )
-    (property "Footprint" "" (id 2) (at 82.2452 45.72 0)
+    (property "Footprint" "Capacitor_SMD:C_0201_0603Metric" (id 2) (at 82.2452 45.72 0)
       (effects (font (size 1.27 1.27)) hide)
     )
@@
       (effects (font (size 1.27 1.27)) (justify right))
     )
-    (property "Footprint" "" (id 2) (at 82.2452 77.47 0)
+    (property "Footprint" "Capacitor_SMD:C_0201_0603Metric" (id 2) (at 82.2452 77.47 0)
       (effects (font (size 1.27 1.27)) hide)
     )
@@
     (property "Reference" "R28" (id 0) (at 168.91 102.87 90))
     (property "Value" "1K" (id 1) (at 168.91 107.95 90))
-    (property "Footprint" "" (id 2) (at 168.91 107.188 90)
+    (property "Footprint" "Resistor_SMD:R_0603_1608Metric" (id 2) (at 168.91 107.188 90)
       (effects (font (size 1.27 1.27)) hide)
     )
@@
       (effects (font (size 1.27 1.27)) (justify left))
     )
-    (property "Footprint" "" (id 2) (at 191.4652 38.1 0)
+    (property "Footprint" "Capacitor_SMD:C_0201_0603Metric" (id 2) (at 191.4652 38.1 0)
       (effects (font (size 1.27 1.27)) hide)
     )
@@
       (effects (font (size 1.27 1.27)) (justify right))
     )
-    (property "Footprint" "" (id 2) (at 124.968 144.78 90)
+    (property "Footprint" "Resistor_SMD:R_0603_1608Metric" (id 2) (at 124.968 144.78 90)
       (effects (font (size 1.27 1.27)) hide)
     )
@@
     )
     (property "Value" "3K 0.05%" (id 1) (at 118.11 138.43 90))
-    (property "Footprint" "" (id 2) (at 118.11 137.668 90)
+    (property "Footprint" "Resistor_SMD:R_0603_1608Metric" (id 2) (at 118.11 137.668 90)
       (effects (font (size 1.27 1.27)) hide)
     )
@@
       (effects (font (size 1.27 1.27)) (justify left))
     )
-    (property "Footprint" "" (id 2) (at 232.7148 68.58 0)
+    (property "Footprint" "Capacitor_SMD:C_0201_0603Metric" (id 2) (at 232.7148 68.58 0)
       (effects (font (size 1.27 1.27)) hide)
     )
@@
       (effects (font (size 1.27 1.27)) (justify right))
     )
-    (property "Footprint" "" (id 2) (at 163.5252 104.14 0)
+    (property "Footprint" "Capacitor_SMD:C_0201_0603Metric" (id 2) (at 163.5252 104.14 0)
       (effects (font (size 1.27 1.27)) hide)
     )
@@
       (effects (font (size 1.27 1.27)) (justify right))
     )
-    (property "Footprint" "" (id 2) (at 150.8252 78.74 0)
+    (property "Footprint" "Capacitor_SMD:C_0201_0603Metric" (id 2) (at 150.8252 78.74 0)
       (effects (font (size 1.27 1.27)) hide)
     )
@@
       (effects (font (size 1.27 1.27)) (justify right))
     )
-    (property "Footprint" "" (id 2) (at 250.698 55.88 90)
+    (property "Footprint" "Resistor_SMD:R_0603_1608Metric" (id 2) (at 250.698 55.88 90)
       (effects (font (size 1.27 1.27)) hide)
     )
@@
       (effects (font (size 1.27 1.27)) (justify left))
     )
-    (property "Footprint" "" (id 2) (at 238.76 38.1 0)
+    (property "Footprint" "TestPoint:TestPoint_Loop_D2.50mm_Drill1.0mm" (id 2) (at 238.76 38.1 0)
       (effects (font (size 1.27 1.27)) hide)
     )
@@
     (property "Reference" "R25" (id 0) (at 168.91 48.26 90))
     (property "Value" "1K" (id 1) (at 168.91 53.34 90))
-    (property "Footprint" "" (id 2) (at 168.91 52.578 90)
+    (property "Footprint" "Resistor_SMD:R_0603_1608Metric" (id 2) (at 168.91 52.578 90)
       (effects (font (size 1.27 1.27)) hide)
     )
@@
     (property "Reference" "U12" (id 0) (at 110.49 39.37 0))
     (property "Value" "ADS131M02IPWR" (id 1) (at 110.49 41.91 0))
-    (property "Footprint" "SOP65P640X120-20N" (id 2) (at 93.98 43.18 0)
+    (property "Footprint" "SamacSys_Parts:SOP65P640X120-20N" (id 2) (at 93.98 43.18 0)
       (effects (font (size 1.27 1.27)) (justify left) hide)
     )
@@
       (effects (font (size 1.27 1.27)) (justify right))
     )
-    (property "Footprint" "" (id 2) (at 163.5252 59.69 0)
+    (property "Footprint" "Capacitor_SMD:C_0201_0603Metric" (id 2) (at 163.5252 59.69 0)
       (effects (font (size 1.27 1.27)) hide)
     )
@@
       (effects (font (size 1.27 1.27)) (justify right))
     )
-    (property "Footprint" "" (id 2) (at 65.7352 143.51 0)
+    (property "Footprint" "Capacitor_SMD:C_0201_0603Metric" (id 2) (at 65.7352 143.51 0)
       (effects (font (size 1.27 1.27)) hide)
     )
@@
       (effects (font (size 1.27 1.27)) (justify left))
     )
-    (property "Footprint" "" (id 2) (at 149.5552 184.15 0)
+    (property "Footprint" "Capacitor_SMD:C_0201_0603Metric" (id 2) (at 149.5552 184.15 0)
       (effects (font (size 1.27 1.27)) hide)
     )
@@
       (effects (font (size 1.27 1.27)) (justify right))
     )
-    (property "Footprint" "" (id 2) (at 143.2052 78.74 0)
-      (effects (font (size 1.27 1.27)) hide)
-    )
+    (property "Footprint" "Capacitor_SMD:C_0201_0603Metric" (id 2) (at 143.2052 78.74 0)
+      (effects (font (size 1.27 1.27)) hide)
+    )
